File: schematics/LED-Lampe Power  ZXLD1374.sch (EAGLE design)
At the start: 50 parts, among them X2 MKDSN1,5/4-5,08, X6 MKDSN1,5/2-5,08

Commit message: - finalized layout - moved to eagle 6.5
Parts:
- added C25: 220µF / 50V Pan FR, rcl:CPOL-EUE5-10.5
- C1: value 470µ / 50V -> 220µF / 50V Pan FR; device rcl:CPOL-EUE5-13 -> rcl:CPOL-EUE5-10.5
- R25, R3, R7, R8, R9: device resistor:R-EU_R1206 -> rcl:R-EU_R1206
- U$1: value FASTON_PIS4728 220µH -> PIS4728 220µH
- U$2, U$3: value FASTON_PIS4728 100µH -> PIS4728 100µH
Connections:
- net +24V: no longer C1.+
- net GND: now also C25.-
- net N$48: now also C25.+
- net N$7: now also C1.+
Other:
- moved on the sheet: C1, C19, C20, C24, C35, D4, D9, JP1, R25, R7, X6-1, X6-2

Commit message: - fix ZXLD1374 case
Parts:
- renumbered U$1 to L$1, U$2 to L$2, U$3 to L$3
Changed lines of the file:
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@@
 <classes>
 <class number="0" name="default" width="0" drill="0">
+<clearance class="0" value="0.2032"/>
 </class>
 </classes>
@@
 <part name="C9" library="resistor" deviceset="C-EU" device="C1206" value="2,2µF / 50V X7R"/>
 <part name="C10" library="resistor" deviceset="C-EU" device="C1206" value="2,2µF / 50V X7R"/>
-<part name="U$2" library="LED-Treiber" deviceset="FASTON_PIS4728" device="" value="PIS4728 100µH"/>
+<part name="L$2" library="LED-Treiber" deviceset="FASTON_PIS4728" device="" value="PIS4728 100µH"/>
 <part name="D2" library="diode" deviceset="MBRS360T3" device="" value="MBRS360T3"/>
 <part name="X6" library="con-phoenix-508" deviceset="MKDSN1,5/2-5,08" device=""/>
@@
 <part name="JP1" library="con-harting-ml" deviceset="ML6" device=""/>
 <part name="+3V2" library="supply1" deviceset="+3V3" device=""/>
-<part name="U$1" library="LED-Treiber" deviceset="FASTON_PIS4728" device="" value="PIS4728 220µH"/>
+<part name="L$1" library="LED-Treiber" deviceset="FASTON_PIS4728" device="" value="PIS4728 220µH"/>
 <part name="U$4" library="LT1676" deviceset="LT1676" device=""/>
 <part name="GND1" library="supply1" deviceset="GND" device=""/>
@@
 <part name="C7" library="resistor" deviceset="C-EU" device="C1206" value="2,2µF / 50V X7R"/>
 <part name="C8" library="resistor" deviceset="C-EU" device="C1206" value="2,2µF / 50V X7R"/>
-<part name="U$3" library="LED-Treiber" deviceset="FASTON_PIS4728" device="" value="PIS4728 100µH"/>
+<part name="L$3" library="LED-Treiber" deviceset="FASTON_PIS4728" device="" value="PIS4728 100µH"/>
 <part name="D1" library="diode" deviceset="MBRS360T3" device="" value="MBRS360T3"/>
 <part name="P+1" library="supply1" deviceset="+24V" device=""/>
@@
 <instance part="C9" gate="G$1" x="261.62" y="38.1"/>
 <instance part="C10" gate="G$1" x="175.26" y="53.34"/>
-<instance part="U$2" gate="G$1" x="251.46" y="27.94"/>
+<instance part="L$2" gate="G$1" x="251.46" y="27.94"/>
 <instance part="D2" gate="G$1" x="241.3" y="38.1" rot="R90"/>
 <instance part="X6" gate="-1" x="116.84" y="-7.62" rot="MR0"/>
@@
 <instance part="JP1" gate="1" x="114.3" y="106.68"/>
 <instance part="+3V2" gate="G$1" x="104.14" y="119.38"/>
-<instance part="U$1" gate="G$1" x="243.84" y="172.72"/>
+<instance part="L$1" gate="G$1" x="243.84" y="172.72"/>
 <instance part="U$4" gate="G$1" x="205.74" y="190.5"/>
 <instance part="GND1" gate="1" x="104.14" y="93.98"/>
@@
 <instance part="C7" gate="G$1" x="261.62" y="116.84"/>
 <instance part="C8" gate="G$1" x="175.26" y="132.08"/>
-<instance part="U$3" gate="G$1" x="251.46" y="106.68"/>
+<instance part="L$3" gate="G$1" x="251.46" y="106.68"/>
 <instance part="D1" gate="G$1" x="241.3" y="116.84" rot="R90"/>
 <instance part="P+1" gate="1" x="137.16" y="142.24"/>
@@
 <wire x1="228.6" y1="172.72" x2="236.22" y2="172.72" width="0.1524" layer="91"/>
 <wire x1="228.6" y1="154.94" x2="228.6" y2="172.72" width="0.1524" layer="91"/>
-<pinref part="U$1" gate="G$1" pin="1"/>
+<pinref part="L$1" gate="G$1" pin="1"/>
 <pinref part="U$4" gate="G$1" pin="V_SW"/>
 <wire x1="218.44" y1="190.5" x2="228.6" y2="190.5" width="0.1524" layer="91"/>
@@
 <wire x1="254" y1="190.5" x2="254" y2="195.58" width="0.1524" layer="91"/>
 <junction x="254" y="190.5"/>
-<pinref part="U$1" gate="G$1" pin="2"/>
+<pinref part="L$1" gate="G$1" pin="2"/>
 <pinref part="U$4" gate="G$1" pin="VCC"/>
 <wire x1="254" y1="195.58" x2="254" y2="203.2" width="0.1524" layer="91"/>
@@
 <pinref part="C9" gate="G$1" pin="2"/>
 <wire x1="261.62" y1="33.02" x2="261.62" y2="27.94" width="0.1524" layer="91"/>
-<pinref part="U$2" gate="G$1" pin="2"/>
+<pinref part="L$2" gate="G$1" pin="2"/>
 <wire x1="259.08" y1="27.94" x2="261.62" y2="27.94" width="0.1524" layer="91"/>
 <pinref part="X2" gate="-3" pin="KL"/>
@@
 <net name="N$17" class="0">
 <segment>
-<pinref part="U$2" gate="G$1" pin="1"/>
+<pinref part="L$2" gate="G$1" pin="1"/>
 <pinref part="U$5" gate="G$1" pin="LX1"/>
 <wire x1="243.84" y1="27.94" x2="241.3" y2="27.94" width="0.1524" layer="91"/>
@@
 <wire x1="261.62" y1="106.68" x2="264.16" y2="106.68" width="0.1524" layer="91"/>
 <wire x1="261.62" y1="111.76" x2="261.62" y2="106.68" width="0.1524" layer="91"/>
-<pinref part="U$3" gate="G$1" pin="2"/>
+<pinref part="L$3" gate="G$1" pin="2"/>
 <wire x1="259.08" y1="106.68" x2="261.62" y2="106.68" width="0.1524" layer="91"/>
 <junction x="261.62" y="106.68"/>
@@
 <net name="N$23" class="0">
 <segment>
-<pinref part="U$3" gate="G$1" pin="1"/>
+<pinref part="L$3" gate="G$1" pin="1"/>
 <pinref part="U$6" gate="G$1" pin="LX1"/>
 <wire x1="243.84" y1="106.68" x2="241.3" y2="106.68" width="0.1524" layer="91"/>
